Commit message: jackal update

File: entities/robots/jackal/urdf/accessories/bridge_plate.urdf.xacro (robot description, xacro)
@@ -1,20 +1,26 @@
 <?xml version="1.0"?>
 <robot xmlns:xacro="http://www.ros.org/wiki/xacro">
-  <xacro:macro name="bridge_plate" params="mount height">
-    <joint name="${mount}_mount_to_${mount}_bridge" type="fixed">
-      <parent link="${mount}_mount"/>
-      <child link="${mount}_bridge"/>
+  <xacro:macro name="bridge_plate" params="prefix parent height *origin">
+    <link name="${prefix}_bridge_base"/>
+    <joint name="${prefix}_bridge_base_joint" type="fixed">
+      <parent link="${parent}"/>
+      <child link="${prefix}_bridge_base" />
+      <xacro:insert_block name="origin" />
+    </joint>
+    <joint name="${prefix}_bridge_joint" type="fixed">
+      <parent link="${prefix}_bridge_base"/>
+      <child link="${prefix}_bridge"/>
       <origin xyz="0.0 0.0 ${height}" rpy="0 0 0"/>
     </joint>
-    <link name="${mount}_bridge">
+    <link name="${prefix}_bridge">
       <visual>
         <origin xyz="0 0 0" rpy="1.5707 0.0 1.5707" />
         <geometry>
-          <mesh filename="package://arena_simulation_setup/entities/robots/jackal/urdf/meshes/bridge-plate.stl"/>
+          <mesh filename="package://jackal_description/meshes/bridge-plate.stl"/>
         </geometry>
         <material name="dark_grey" />
       </visual>
     </link>
-    <standoff_box mount="${mount}" height="${height}" />
+    <xacro:standoff_box prefix="${prefix}" parent="${prefix}_bridge_base" height="${height}" />
   </xacro:macro>
 </robot>

File: entities/robots/jackal/urdf/accessories/camera_mount.urdf.xacro (robot description, xacro)
@@ -5,5 +5,5 @@
         <origin xyz="0 0 0" rpy="1.5707 0 1.5707" />
         <geometry>
-          <mesh filename="package://arena_simulation_setup/entities/robots/jackal/urdf/meshes/camera-bracket.stl" scale="0.001 0.001 0.001" />
+          <mesh filename="package://jackal_description/meshes/camera-bracket.stl" scale="0.001 0.001 0.001" />
         </geometry>
         <material name="dark_grey" />
@@ -14,5 +14,5 @@
         <origin xyz="0 0 0" rpy="0 0 1.5707" />
         <geometry>
-          <mesh filename="package://arena_simulation_setup/entities/robots/jackal/urdf/meshes/camera-beam.stl" scale="0.001 0.001 0.001" />
+          <mesh filename="package://jackal_description/meshes/camera-beam.stl" scale="0.001 0.001 0.001" />
         </geometry>
         <material name="dark_grey" />

File: entities/robots/jackal/urdf/accessories/hokuyo_utm30.urdf.xacro (robot description, xacro)
@@ -1,14 +1,17 @@
 <?xml version="1.0"?>
 <robot xmlns:xacro="http://ros.org/wiki/xacro">
-  <xacro:macro name="hokuyo_ust10_mount" params="prefix topic parent_link *origin">
-    <xacro:macro name="hokuyo_ust10" params="frame:=laser topic:=scan sample_size:=720 update_rate:=50
-               min_angle:=-2.35619 max_angle:=2.35619 min_range:=0.1 max_range:=30.0 robot_namespace:=/">
+  <xacro:macro name="hokuyo_utm30_mount" params="prefix topic parent_link min_angle:=-2.2689  max_angle:=2.2689 *origin">
+    <xacro:macro name="hokuyo_utm30" params="frame:=laser topic:=scan sample_size:=1440 update_rate:=50
+               min_angle:=-2.2689 max_angle:=2.2689 min_range:=0.1 max_range:=30.0 robot_namespace:=/">
+      <xacro:property name="mass" value="0.370"/>
+      <xacro:property name="base" value="0.06" />
+      <xacro:property name="height" value="0.087"/>
       <link name="${frame}">
         <inertial>
-          <mass value="1.1" />
+          <mass value="${mass}" />
           <origin xyz="0 0 0" />
-          <inertia ixx="${0.0833333 * 1.1 * (0.102*0.102 + 0.152*0.152)}" ixy="0.0" ixz="0.0"
-            iyy="${0.0833333 * 1.1 * (0.105*0.105 + 0.152*0.152)}" iyz="0.0"
-            izz="${0.0833333 * 1.1 * (0.105*0.105 + 0.102*0.102)}" />
+          <inertia ixx="${mass/12 * (base*base + height*height)}" ixy="0.0" ixz="0.0"
+                   iyy="${mass/12 * (base*base + height*height)}" iyz="0.0"
+                   izz="${mass/12 * 2 * (base * base)}" />
         </inertial>
       </link>
@@ -39,16 +42,13 @@
             </noise>
           </ray>
-          <plugin name="gazebo_ros_laser" filename="libgazebo_ros_ray_sensor.so">
-            <ros>
-              <namespace>${robot_namespace}</namespace>
-              <remapping>~/out:=${topic}</remapping>
-            </ros>
-            <output_type>sensor_msgs/LaserScan</output_type>
-            <frame_name>${frame}</frame_name>
+          <plugin name="gazebo_ros_laser" filename="libgazebo_ros_laser.so">
+            <topicName>${topic}</topicName>
+            <frameName>${frame}</frameName>
+            <robotNamespace>${robot_namespace}</robotNamespace>
           </plugin>
         </sensor>
       </gazebo>
     </xacro:macro>
-    <xacro:hokuyo_ust10 frame="${prefix}_laser" topic="${topic}"/>
+    <xacro:hokuyo_utm30 frame="${prefix}_laser" topic="${topic}"/>
     <joint name="${prefix}_laser_mount_joint" type="fixed">
       <xacro:insert_block name="origin" />
@@ -61,5 +61,5 @@
         <geometry>
           <!-- Origin of this mesh is the base of the bracket. -->
-          <mesh filename="package://jackal_description/meshes/hokuyo_ust10.stl" />
+          <mesh filename="package://jackal_description/meshes/hokuyo_utm30.stl" />
         </geometry>
         <material name="dark_grey" />
@@ -68,5 +68,5 @@
     <joint name="${prefix}_laser_joint" type="fixed">
       <!-- This offset is from the base of the bracket to the LIDAR's focal point. -->
-      <origin xyz="0 0 0.0474" rpy="0 0 0" />
+      <origin xyz="0 0 0.055" rpy="0 0 0" />
       <parent link="${prefix}_laser_mount" />
       <child link="${prefix}_laser" />

File: entities/robots/jackal/urdf/accessories/novatel_smart6.urdf.xacro (robot description, xacro)
@@ -6,5 +6,5 @@
       <origin xyz="0 0 0" rpy="0 0 0" />
       <geometry>
-        <mesh filename="package://arena_simulation_setup/entities/robots/jackal/urdf/meshes/novatel-smart6.stl"/>
+        <mesh filename="package://jackal_description/meshes/novatel-smart6.stl"/>
       </geometry>
       <material name="novatel_white">

File: entities/robots/jackal/urdf/accessories/sick_lms1xx_upright_mount.urdf.xacro (robot description, xacro)
@@ -27,5 +27,5 @@
 <robot xmlns:xacro="http://www.ros.org/wiki/xacro">
   <xacro:include filename="$(find lms1xx)/urdf/sick_lms1xx.urdf.xacro" />
-  <xacro:macro name="sick_lms1xx_mount" params="prefix topic parent_link *origin">
+  <xacro:macro name="sick_lms1xx_upright_mount" params="prefix topic parent_link *origin">
     <xacro:sick_lms1xx frame="${prefix}_laser" topic="${topic}" />
     <joint name="${prefix}_laser_mount_joint" type="fixed">
@@ -39,5 +39,5 @@
         <geometry>
           <!-- Origin of this mesh is the base of the bracket. -->
-          <mesh filename="package://jackal_description/meshes/sick-lms1xx-bracket.stl" />
+          <mesh filename="package://jackal_description/meshes/sick-lms1xx-upright-bracket.stl" />
         </geometry>
         <material name="dark_grey" />

File: entities/robots/jackal/urdf/accessories/stereo_camera_mount.urdf.xacro (robot description, xacro)
@@ -6,5 +6,5 @@
         <origin xyz="0 0 0" rpy="0 0 0" />
         <geometry>
-          <mesh filename="package://arena_simulation_setup/entities/robots/jackal/urdf/meshes/stereo-camera-bracket.stl" />
+          <mesh filename="package://jackal_description/meshes/stereo-camera-bracket.stl" />
         </geometry>
         <material name="dark_grey" />
@@ -15,5 +15,5 @@
         <origin xyz="0 0 0" rpy="0 0 0" />
         <geometry>
-          <mesh filename="package://arena_simulation_setup/entities/robots/jackal/urdf/meshes/stereo-camera-beam.stl" />
+          <mesh filename="package://jackal_description/meshes/stereo-camera-beam.stl" />
         </geometry>
         <material name="dark_grey" />

File: entities/robots/jackal/urdf/jackal.urdf.xacro (robot description, xacro)
@@ -1,4 +1,7 @@
 <?xml version="1.0"?>
 <robot name="jackal" xmlns:xacro="http://www.ros.org/wiki/xacro">
+  <xacro:arg name="is_sim" default="false" />
+  <xacro:arg name="prefix" default="" />
+  <xacro:arg name="gazebo_controllers" default="$(find jackal_control)/config/control.yaml" />
   <xacro:property name="PI" value="3.1415926535897931" />
   <xacro:property name="wheelbase" value="0.262" />
@@ -22,5 +25,5 @@
         <origin xyz="0 0 0" rpy="${PI/2} 0 0"/>
         <geometry>
-          <mesh filename="package://arena_simulation_setup/entities/robots/jackal/urdf/meshes/jackal-wheel.stl"/>
+          <mesh filename="package://jackal_description/meshes/jackal-wheel.stl"/>
         </geometry>
         <material name="black" />
@@ -50,5 +53,5 @@
       <fdir1 value="1 0 0"/>
     </gazebo>
-    <joint name="${prefix}_wheel" type="continuous">
+    <joint name="${prefix}_wheel_joint" type="continuous">
       <parent link="chassis_link"/>
       <child link="${prefix}_wheel_link" />
@@ -90,5 +93,5 @@
       <origin xyz="0 0 ${footprint_vertical_offset}" rpy="${PI/2} 0 ${PI/2}"/>
       <geometry>
-        <mesh filename="package://arena_simulation_setup/entities/robots/jackal/urdf/meshes/jackal-base.stl"/>
+        <mesh filename="package://jackal_description/meshes/jackal-base.stl"/>
       </geometry>
       <material name="dark_grey" />
@@ -115,5 +118,5 @@
       <visual>
         <geometry>
-          <mesh filename="package://arena_simulation_setup/entities/robots/jackal/urdf/meshes/jackal-fender.stl"/>
+          <mesh filename="package://jackal_description/meshes/jackal-fender.stl"/>
         </geometry>
         <material name="yellow" />
@@ -125,5 +128,5 @@
       <visual>
         <geometry>
-          <mesh filename="package://arena_simulation_setup/entities/robots/jackal/urdf/meshes/accessory_fender.stl"/>
+          <mesh filename="package://jackal_description/meshes/accessory_fender.stl"/>
         </geometry>
         <material name="yellow" />
@@ -146,5 +149,5 @@
       <visual>
         <geometry>
-          <mesh filename="package://arena_simulation_setup/entities/robots/jackal/urdf/meshes/jackal-fender.stl"/>
+          <mesh filename="package://jackal_description/meshes/jackal-fender.stl"/>
         </geometry>
         <material name="yellow" />
@@ -156,5 +159,5 @@
       <visual>
         <geometry>
-          <mesh filename="package://arena_simulation_setup/entities/robots/jackal/urdf/meshes/accessory_fender.stl"/>
+          <mesh filename="package://jackal_description/meshes/accessory_fender.stl"/>
         </geometry>
         <material name="yellow" />
@@ -213,5 +216,5 @@
     <parent link="mid_mount" />
     <child link="rear_mount" />
-    <origin xyz="${mount_spacing} 0 0" />
+    <origin xyz="${-mount_spacing} 0 0" />
   </joint>
   <link name="front_mount"></link>
@@ -219,12 +222,46 @@
     <parent link="mid_mount" />
     <child link="front_mount" />
-    <origin xyz="${-mount_spacing} 0 0" rpy="0 0 0" />
-  </joint>
+    <origin xyz="${mount_spacing} 0 0" />
+  </joint>
+  <!-- ROS2 controls -->
+  <ros2_control name="jackal_hardware" type="system">
+    <hardware>
+      <xacro:if value="$(arg is_sim)">
+        <plugin>gazebo_ros2_control/GazeboSystem</plugin>
+      </xacro:if>
+      <xacro:unless value="$(arg is_sim)">
+        <plugin>jackal_hardware/JackalHardware</plugin>
+        <plugin>fake_components/GenericSystem</plugin>
+      </xacro:unless>
+    </hardware>
+    <joint name="front_left_wheel_joint">
+      <command_interface name="velocity"/>
+      <state_interface name="position"/>
+      <state_interface name="velocity"/>
+    </joint>
+    <joint name="rear_left_wheel_joint">
+      <command_interface name="velocity"/>
+      <state_interface name="position"/>
+      <state_interface name="velocity"/>
+    </joint>
+    <joint name="front_right_wheel_joint">
+      <command_interface name="velocity"/>
+      <state_interface name="position"/>
+      <state_interface name="velocity"/>
+    </joint>
+    <joint name="rear_right_wheel_joint">
+      <command_interface name="velocity"/>
+      <state_interface name="position"/>
+      <state_interface name="velocity"/>
+    </joint>
+  </ros2_control>
   <!-- Bring in simulation data for Gazebo. -->
-  <xacro:include filename="$(find arena_simulation_setup)/entities/robots/jackal/urdf/jackal.gazebo" />
+  <xacro:if value="$(arg is_sim)">
+    <xacro:include filename="$(find jackal_description)/urdf/jackal.gazebo" />
+  </xacro:if>
   <!-- Optional standard accessories, including their simulation data. The rendering
        of these into the final description is controlled by optenv variables, which
        default each one to off.-->
-  <xacro:include filename="$(find arena_simulation_setup)/entities/robots/jackal/urdf/accessories.urdf.xacro" />
+  <xacro:include filename="$(find jackal_description)/urdf/accessories.urdf.xacro" />
   <!-- Optional custom includes. -->
   <xacro:include filename="$(optenv JACKAL_URDF_EXTRAS empty.urdf)" />
