Commit message: add turtlebot nav2 functionality

File: entities/robots/turtlebot/urdf/sensors/rplidar.urdf.xacro (robot description, xacro)
@@ -41,4 +41,10 @@
             <max_angle>3.14159</max_angle>
           </horizontal>
+          <vertical>
+            <samples>16</samples>
+            <resolution>1</resolution>
+            <min_angle>-0.261799</min_angle>
+            <max_angle>0.261799</max_angle>
+          </vertical>
         </scan>
         <range>
@@ -48,8 +54,7 @@
         </range>
       </lidar>
-      <always_on>true</always_on>
+      <always_on>1</always_on>
       <visualize>true</visualize>
     </sensor>
-    <material>Gazebo/DarkGrey</material>
   </gazebo>
   <gazebo reference="${name}_joint">
