Commit message: update urdfs and launch files

File: entities/robots/turtlebot/urdf/sensors/oakd.urdf.xacro (robot description, xacro)
@@ -97,4 +97,70 @@
       <origin xyz="0 0 0" rpy="-${M_PI/2} 0 -${M_PI/2}" />
   </joint>
+  <gazebo reference="${name}_imu_joint">
+    <sensor name="imu_sensor" type="imu">
+      <plugin filename="libgz-sim-imu-system" name="gz::sim::systems::Imu">
+        <topic>/imu/data</topic>
+        <frame_id>${name}_imu_frame</frame_id>
+      </plugin>
+      <always_on>true</always_on>
+      <update_rate>100</update_rate>
+      <visualize>true</visualize>
+      <imu>
+        <angular_velocity>
+          <x>
+            <noise type="gaussian">
+              <mean>0.0</mean>
+              <stddev>2e-4</stddev>
+              <bias_mean>0.0000075</bias_mean>
+              <bias_stddev>0.0000008</bias_stddev>
+            </noise>
+          </x>
+          <y>
+            <noise type="gaussian">
+              <mean>0.0</mean>
+              <stddev>2e-4</stddev>
+              <bias_mean>0.0000075</bias_mean>
+              <bias_stddev>0.0000008</bias_stddev>
+            </noise>
+          </y>
+          <z>
+            <noise type="gaussian">
+              <mean>0.0</mean>
+              <stddev>2e-4</stddev>
+              <bias_mean>0.0000075</bias_mean>
+              <bias_stddev>0.0000008</bias_stddev>
+            </noise>
+          </z>
+        </angular_velocity>
+        <linear_acceleration>
+          <x>
+            <noise type="gaussian">
+              <mean>0.0</mean>
+              <stddev>1.7e-2</stddev>
+              <bias_mean>0.1</bias_mean>
+              <bias_stddev>0.001</bias_stddev>
+            </noise>
+          </x>
+          <y>
+            <noise type="gaussian">
+              <mean>0.0</mean>
+              <stddev>1.7e-2</stddev>
+              <bias_mean>0.1</bias_mean>
+              <bias_stddev>0.001</bias_stddev>
+            </noise>
+          </y>
+          <z>
+            <noise type="gaussian">
+              <mean>0.0</mean>
+              <stddev>1.7e-2</stddev>
+              <bias_mean>0.1</bias_mean>
+              <bias_stddev>0.001</bias_stddev>
+            </noise>
+          </z>
+        </linear_acceleration>
+      </imu>
+    </sensor>
+    <material>Gazebo/Grey</material>
+  </gazebo>
   <!-- Gazebo links and joints -->
   <gazebo reference="${name}_rgb_camera_frame">

File: entities/robots/turtlebot/urdf/sensors/rplidar.urdf.xacro (robot description, xacro)
@@ -10,5 +10,12 @@
   <xacro:property name="collision_y_offset"       value="${1.3*cm2m}" />
   <xacro:property name="collision_z_offset"       value="${-1.9*cm2m}" />
-  <joint name="${name}_joint" type="fixed">
+  <plugin
+    filename="gz-sim-joint-state-publisher-system"
+    name="gz::sim::systems::JointStatePublisher">
+    <topic>joint_states</topic>
+    <joint_name>wheel_left_link</joint_name>
+    <joint_name>wheel_right_link</joint_name>
+  </plugin>
+  <joint name="rplidar_joint" type="fixed">
     <parent link="${parent_link}"/>
     <child link="${name}_link"/>
@@ -59,6 +66,17 @@
     </sensor>
   </gazebo>
-  <gazebo reference="${name}_joint">
-    <preserveFixedJoint>true</preserveFixedJoint>
+  <gazebo reference="wheel_left_link">
+    <mu1>0.8</mu1>
+    <mu2>0.8</mu2>
+    <fdir1>1 0 0</fdir1>
+    <kp>1000000.0</kp>
+    <kd>100.0</kd>
+  </gazebo>
+  <gazebo reference="wheel_right_link">
+    <mu1>0.8</mu1>
+    <mu2>0.8</mu2>
+    <fdir1>1 0 0</fdir1>
+    <kp>1000000.0</kp>
+    <kd>100.0</kd>
   </gazebo>
 </xacro:macro>

File: entities/robots/turtlebot/urdf/turtlebot.urdf.xacro (robot description, xacro)
@@ -1,4 +1,4 @@
 <?xml version="1.0"?>
-<robot name="turtlebot4" xmlns:xacro="http://ros.org/wiki/xacro">
+<robot name="turtlebot" xmlns:xacro="http://ros.org/wiki/xacro">
   <!-- Base create3 model -->
   <xacro:include filename="$(find irobot_create_description)/urdf/create3.urdf.xacro">
@@ -40,4 +40,5 @@
     <child link="shell_link"/>
     <origin xyz="0 0 ${shell_z_offset}" rpy="0 0 0"/>
+    <turnGravityOff>false</turnGravityOff>
   </joint>
   <link name="shell_link">
@@ -58,7 +59,9 @@
                iyy="0.00164666421" iyz="0.00000564466" izz="0.00424540124" />
     </inertial>
+    <turnGravityOff>false</turnGravityOff>
   </link>
   <gazebo reference="shell_link">
     <material>Gazebo/Black</material>
+    <turnGravityOff>false</turnGravityOff>
   </gazebo>
   <!-- Weight Blocks -->
@@ -112,6 +115,4 @@
       <wheel_radius>0.098</wheel_radius>
       <odom_publish_frequency>50</odom_publish_frequency>
-      <base_frame_id>base_link</base_frame_id>
-      <odom_frame_id>odom</odom_frame_id>
       <publish_odom>true</publish_odom>
       <publish_odom_tf>true</publish_odom_tf>
