Commit message: 保留对 dingo 文件的修改

File: entities/robots/dingo/urdf/accessories/intel_realsense.urdf.xacro (robot description, xacro)
@@ -5,12 +5,54 @@
   gazebo plugin to simulate data from the camera
 -->
+<!-- IMPORTANT NOTE FOR MULTIPLE REALSENSES:
+  As of Sept. 2022, due to limitations with the 'realsense2_description' package
+  (see realsense2_description/urdf/_materials.xacro.urdf):
+    1. the include parameter must be set to FALSE, and
+    2. the following files must be included in the parent xacro file that will
+        include this one:
+  '''
+  <xacro:if value="${rs_model == 'd435'}">
+    <xacro:include filename="$(find realsense2_description)/urdf/_d435.urdf.xacro" />
+  </xacro:if>
+  <xacro:if value="${rs_model == 'd435i'}">
+    <xacro:include filename="$(find realsense2_description)/urdf/_d435i.urdf.xacro" />
+  </xacro:if>
+  <xacro:if value="${rs_model == 'd415'}">
+    <xacro:include filename="$(find realsense2_description)/urdf/_d415.urdf.xacro" />
+  </xacro:if>
+  <xacro:if value="${rs_model == 'd455'}">
+    <xacro:include filename="$(find realsense2_description)/urdf/_d435.urdf.xacro" />
+  </xacro:if>
+  '''
+  Multiple inclusions of any of these files (even when namespaced), will define
+  the materials at a global level, violating uniqueness property of xacro materials.
+  Therefore, it is not possible at this time to have different models of Realsense
+  cameras on the same URDF, without modifying the `realsense2_description` package.
+ -->
 <robot xmlns:xacro="http://ros.org/wiki/xacro">
   <xacro:macro name="realsense_sensor" params="
                rs_model:=d435
                prefix:=front
+               parent:=front_mount
                topic:=realsense
                width:=680
                height:=480
-               update_rate:=30">
+               update_rate:=30
+               include:=1
+               *origin">
+    <xacro:if value="${include}">
+      <xacro:if value="${rs_model == 'd435'}">
+        <xacro:include filename="$(find realsense2_description)/urdf/_d435.urdf.xacro" />
+      </xacro:if>
+      <xacro:if value="${rs_model == 'd435i'}">
+        <xacro:include filename="$(find realsense2_description)/urdf/_d435i.urdf.xacro" />
+      </xacro:if>
+      <xacro:if value="${rs_model == 'd415'}">
+        <xacro:include filename="$(find realsense2_description)/urdf/_d415.urdf.xacro" />
+      </xacro:if>
+      <xacro:if value="${rs_model == 'd455'}">
+        <xacro:include filename="$(find realsense2_description)/urdf/_d435.urdf.xacro" />
+      </xacro:if>
+    </xacro:if>
     <xacro:macro name="realsense_gazebo" params="
               prefix=front              model=d4
@@ -20,5 +62,5 @@
               width:=640                height:=480
               update_rate:=30
-              robot_namespace:=/">
+              namespace:=/">
      <!--
        The gazebo plugin aligns the depth data with the Z axis, with X=left and Y=up
@@ -80,8 +122,7 @@
     </xacro:macro>
     <xacro:if value="${rs_model == 'd435'}">
-      <xacro:include filename="$(find realsense2_description)/urdf/_d435.urdf.xacro" />
-      <xacro:sensor_d435 parent="${prefix}_mount"
+      <xacro:sensor_d435 parent="${parent}"
                         name="${prefix}_realsense">
-        <origin xyz="$(optenv DINGO_REALSENSE_OFFSET 0 0 0)" rpy="$(optenv DINGO_REALSENSE_RPY 0 0 0)" />
+        <xacro:insert_block name="origin"/>
       </xacro:sensor_d435>
       <xacro:realsense_gazebo
@@ -98,13 +139,12 @@
     </xacro:if>
     <xacro:if value="${rs_model == 'd435i'}">
-      <xacro:include filename="$(find realsense2_description)/urdf/_d435i.urdf.xacro" />
-      <xacro:sensor_d435i parent="$(optenv DINGO_REALSENSE_MOUNT front)_mount"
-                          name="$(optenv DINGO_REALSENSE_MOUNT front)_realsense">
-        <origin xyz="$(optenv DINGO_REALSENSE_OFFSET 0 0 0)" rpy="$(optenv DINGO_REALSENSE_RPY 0 0 0)" />
+      <xacro:sensor_d435i parent="${parent}"
+                          name="${prefix}_realsense">
+        <xacro:insert_block name="origin"/>
       </xacro:sensor_d435i>
       <xacro:realsense_gazebo
-         prefix="$(optenv DINGO_REALSENSE_MOUNT front)"
-         frame="$(optenv DINGO_REALSENSE_MOUNT front)_realsense_link"
-         topic="$(optenv DINGO_REALSENSE_TOPIC realsense)"
+         prefix="${prefix}"
+         frame="${prefix}_realsense_link"
+         topic="${topic}"
          h_fov="1.5184351666666667"
          v_fov="1.0122901111111111"
@@ -123,6 +163,6 @@
           <robotNamespace>/</robotNamespace>
           <updateRate>30.0</updateRate>
-          <bodyName>$(optenv DINGO_REALSENSE_MOUNT front)_realsense_link</bodyName>
-          <topicName>$(optenv DINGO_REALSENSE_TOPIC realsense)/accel/sample</topicName>
+          <bodyName>${prefix}_realsense_link</bodyName>
+          <topicName>${topic}/accel/sample</topicName>
           <accelDrift>0.005 0.005 0.005</accelDrift>
           <accelGaussianNoise>0.005 0.005 0.005</accelGaussianNoise>
@@ -135,6 +175,6 @@
           <robotNamespace>/</robotNamespace>
           <updateRate>30.0</updateRate>
-          <bodyName>$(optenv DINGO_REALSENSE_MOUNT front)_realsense_link</bodyName>
-          <topicName>$(optenv DINGO_REALSENSE_TOPIC realsense)/gyro/sample</topicName>
+          <bodyName>${prefix}_realsense_link</bodyName>
+          <topicName>${topic}/gyro/sample</topicName>
           <accelDrift>0.005 0.005 0.005</accelDrift>
           <accelGaussianNoise>0.005 0.005 0.005</accelGaussianNoise>
@@ -147,13 +187,12 @@
     </xacro:if>
     <xacro:if value="${rs_model == 'd415'}">
-      <xacro:include filename="$(find realsense2_description)/urdf/_d415.urdf.xacro" />
-      <xacro:sensor_d415 parent="$(optenv DINGO_REALSENSE_MOUNT front)_mount"
-                         name="$(optenv DINGO_REALSENSE_MOUNT front)_realsense">
-        <origin xyz="$(optenv DINGO_REALSENSE_OFFSET 0 0 0)" rpy="$(optenv DINGO_REALSENSE_RPY 0 0 0)" />
+      <xacro:sensor_d415 parent="${parent}"
+                         name="${prefix}_realsense">
+        <xacro:insert_block name="origin"/>
       </xacro:sensor_d415>
       <xacro:realsense_gazebo
-         prefix="$(optenv DINGO_REALSENSE_MOUNT front)"
-         frame="$(optenv DINGO_REALSENSE_MOUNT front)_realsense_link"
-         topic="$(optenv DINGO_REALSENSE_TOPIC realsense)"
+         prefix="${prefix}"
+         frame="${prefix}_realsense_link"
+         topic="${topic}"
          h_fov="1.1344640137963142"
          v_fov="0.6981317007977318"
@@ -166,13 +205,12 @@
     <xacro:if value="${rs_model == 'd455'}">
       <!-- TODO: not officially supported yet. Use the D435 mesh for now, even though it's the wrong size -->
-      <xacro:include filename="$(find realsense2_description)/urdf/_d435.urdf.xacro" />
-      <xacro:sensor_d435 parent="$(optenv DINGO_REALSENSE_MOUNT front)_mount"
-                         name="$(optenv DINGO_REALSENSE_MOUNT front)_realsense">
-        <origin xyz="$(optenv DINGO_REALSENSE_OFFSET 0 0 0)" rpy="$(optenv DINGO_REALSENSE_RPY 0 0 0)" />
+      <xacro:sensor_d435 parent="${parent}"
+                         name="${prefix}_realsense">
+        <xacro:insert_block name="origin"/>
       </xacro:sensor_d435>
       <xacro:realsense_gazebo
-         prefix="$(optenv DINGO_REALSENSE_MOUNT front)"
-         frame="$(optenv DINGO_REALSENSE_MOUNT front)_realsense_link"
-         topic="$(optenv DINGO_REALSENSE_TOPIC realsense)"
+         prefix="${prefix}"
+         frame="${prefix}_realsense_link"
+         topic="${topic}"
          h_fov="1.5009831567151233"
          v_fov="0.9948376736367678"
@@ -221,12 +259,12 @@
       </joint>
       <joint type="fixed" name="${prefix}_realsense_mount_joint">
-        <parent link="${prefix}_mount" />
+        <parent link="${parent}" />
         <child link="${prefix}_realsense_bottom_screw_frame" />
         <origin xyz="0 0 0.004" rpy="0 0 0" />
       </joint>
       <xacro:realsense_gazebo
-         prefix="$(optenv DINGO_REALSENSE_MOUNT front)"
-         frame="$(optenv DINGO_REALSENSE_MOUNT front)_realsense_link"
-         topic="$(optenv DINGO_REALSENSE_TOPIC realsense)"
+         prefix="${prefix}"
+         frame="${prefix}_realsense_link"
+         topic="${topic}"
          h_fov="1.2217304763960306"
          v_fov="0.9599310885968813"

File: entities/robots/dingo/urdf/dingo-d.urdf.xacro (robot description, xacro)
@@ -1,4 +1,5 @@
 <?xml version="1.0"?>
 <robot name="dingo" xmlns:xacro="http://www.ros.org/wiki/xacro">
+  <xacro:property name="pacs_enabled" value="$(optenv DINGO_PACS_ENABLED 0)"/>
   <xacro:property name="PI" value="3.1415926535897931" />
   <xacro:property name="wheel_radius" value="0.049" />
@@ -18,5 +19,5 @@
         <origin xyz="0 0 0" rpy="0 0 0"/>
         <geometry>
-          <mesh filename="file://$(find arena_simulation_setup)/entities/robots/dingo/meshes/wheel.stl"/>
+          <mesh filename="package://arena_simulation_setup/entities/robots/dingo/meshes/wheel.stl"/>
         </geometry>
         <material name="black" />
@@ -74,5 +75,5 @@
         <sphere radius="0.01"/>
       </geometry>
-      <material name="Black"/>
+      <material name="black"/>
     </visual>
     <collision>
@@ -106,5 +107,5 @@
   </joint>
   <gazebo reference="rear_caster">
-    <turnGravityOff>true</turnGravityOff>
+    <turnGravityOff>false</turnGravityOff>
     <kp>1000000.0</kp>
     <kd>100.0</kd>
@@ -125,5 +126,5 @@
       <origin xyz="0 0 0" rpy="0 0 0"/>
       <geometry>
-        <mesh filename="file://$(find arena_simulation_setup)/entities/robots/dingo/meshes/diff_chassis.dae"/>
+        <mesh filename="package://arena_simulation_setup/entities/robots/dingo/meshes/diff_chassis.dae"/>
       </geometry>
     </visual>
@@ -131,5 +132,5 @@
       <origin xyz="0 0 0"/>
       <geometry>
-        <mesh filename="file://$(find arena_simulation_setup)/entities/robots/dingo/meshes/diff_chassis_collision.stl"/>
+        <mesh filename="package://arena_simulation_setup/entities/robots/dingo/meshes/diff_chassis_collision.stl"/>
       </geometry>
     </collision>
@@ -138,5 +139,9 @@
       <origin xyz="0 0 0" rpy="0 0 0"/>
       <mass value="10.0"/>
-      <inertia  ixx="0.2216" ixy="0" ixz="0"  iyy="0.2458" iyz="0"  izz="0.4474"/>
+      <!-- Moments of inertia: ( chassis without wheels ) -->
+      <inertia
+        ixx="0.2216" ixy="0" ixz="0"
+        iyy="0.2458" iyz="0"
+        izz="0.4474"/>
       </inertial>
   </link>
@@ -164,40 +169,42 @@
       - rear
   -->
-  <link name="front_mount"/>
-  <link name="front_b_mount"/>
-  <link name="front_c_mount"/>
-  <link name="rear_mount"/>
-  <link name="rear_b_mount"/>
-  <link name="rear_c_mount"/>
-  <joint name="front_c_mount_joint" type="fixed">
-    <origin xyz="0.040 0 0.064263" rpy="0 0 0" />
-    <parent link="chassis_link"/>
-    <child link="front_c_mount" />
-  </joint>
-  <joint name="front_b_mount_joint" type="fixed">
-    <origin xyz="0.080 0 0" rpy="0 0 0" />
-    <parent link="front_c_mount"/>
-    <child link="front_b_mount" />
-  </joint>
-  <joint name="front_mount_joint" type="fixed">
-    <origin xyz="0.080 0 0" rpy="0 0 0" />
-    <parent link="front_b_mount"/>
-    <child link="front_mount" />
-  </joint>
-  <joint name="rear_c_mount_joint" type="fixed">
-    <origin xyz="-0.040 0 0.064263" rpy="0 0 0" />
-    <parent link="chassis_link"/>
-    <child link="rear_c_mount" />
-  </joint>
-  <joint name="rear_b_mount_joint" type="fixed">
-    <origin xyz="-0.080 0 0" rpy="0 0 0" />
-    <parent link="rear_c_mount"/>
-    <child link="rear_b_mount" />
-  </joint>
-  <joint name="rear_moint_joint" type="fixed">
-    <origin xyz="-0.080 0 0" rpy="0 0 0" />
-    <parent link="rear_b_mount"/>
-    <child link="rear_mount" />
-  </joint>
+  <xacro:unless value="${pacs_enabled}">
+    <link name="front_mount"/>
+    <link name="front_b_mount"/>
+    <link name="front_c_mount"/>
+    <link name="rear_mount"/>
+    <link name="rear_b_mount"/>
+    <link name="rear_c_mount"/>
+    <joint name="front_c_mount_joint" type="fixed">
+      <origin xyz="0.040 0 0.064263" rpy="0 0 0" />
+      <parent link="chassis_link"/>
+      <child link="front_c_mount" />
+    </joint>
+    <joint name="front_b_mount_joint" type="fixed">
+      <origin xyz="0.080 0 0" rpy="0 0 0" />
+      <parent link="front_c_mount"/>
+      <child link="front_b_mount" />
+    </joint>
+    <joint name="front_mount_joint" type="fixed">
+      <origin xyz="0.080 0 0" rpy="0 0 0" />
+      <parent link="front_b_mount"/>
+      <child link="front_mount" />
+    </joint>
+    <joint name="rear_c_mount_joint" type="fixed">
+      <origin xyz="-0.040 0 0.064263" rpy="0 0 0" />
+      <parent link="chassis_link"/>
+      <child link="rear_c_mount" />
+    </joint>
+    <joint name="rear_b_mount_joint" type="fixed">
+      <origin xyz="-0.080 0 0" rpy="0 0 0" />
+      <parent link="rear_c_mount"/>
+      <child link="rear_b_mount" />
+    </joint>
+    <joint name="rear_moint_joint" type="fixed">
+      <origin xyz="-0.080 0 0" rpy="0 0 0" />
+      <parent link="rear_b_mount"/>
+      <child link="rear_mount" />
+    </joint>
+  </xacro:unless>
   <!--
     Mounting point for accessories on the front bumper.
@@ -211,4 +218,7 @@
     <child link="front_bumper_mount" />
   </joint>
+  <!-- PACS -->
+  <xacro:include filename="$(find arena_simulation_setup)/entities/robots/dingo/urdf/pacs.urdf.xacro"/>
+  <xacro:pacs/>
   <!-- Bring in simulation data for Gazebo. -->
   <xacro:include filename="$(find arena_simulation_setup)/entities/robots/dingo/urdf/dingo.gazebo" />
@@ -218,4 +228,4 @@
   <xacro:include filename="$(find arena_simulation_setup)/entities/robots/dingo/urdf/accessories.urdf.xacro" />
   <!-- Optional custom includes. -->
-  <!--<xacro:include filename="$(optenv DINGO_URDF_EXTRAS empty.urdf)" />-->
+  <xacro:include filename="$(optenv DINGO_URDF_EXTRAS empty.urdf)" />
 </robot>

File: entities/robots/dingo/urdf/dingo-o.urdf.xacro (robot description, xacro)
@@ -1,4 +1,5 @@
 <?xml version="1.0"?>
 <robot name="dingo" xmlns:xacro="http://www.ros.org/wiki/xacro">
+  <xacro:property name="pacs_enabled" value="$(optenv DINGO_PACS_ENABLED 0)" />
   <xacro:property name="PI" value="3.1415926535897931" />
   <xacro:property name="wheelbase" value="0.570" />
@@ -75,5 +76,5 @@
       <origin xyz="0 0 0" rpy="0 0 0"/>
       <geometry>
-        <mesh filename="file://$(find arena_simulation_setup)/entities/robots/dingo/meshes/omni_chassis.dae"/>
+        <mesh filename="package://arena_simulation_setup/entities/robots/dingo/meshes/omni_chassis.dae"/>
       </geometry>
       <material name="dark_grey" />
@@ -82,5 +83,5 @@
       <origin xyz="0 0 0"/>
       <geometry>
-        <mesh filename="file://$(find arena_simulation_setup)/entities/robots/dingo/meshes/omni_chassis_collision.stl"/>
+        <mesh filename="package://arena_simulation_setup/entities/robots/dingo/meshes/omni_chassis_collision.stl"/>
       </geometry>
     </collision>
@@ -89,5 +90,9 @@
       <origin xyz="0 0 0" rpy="0 0 0"/>
       <mass value="14"/>
-      <inertia  ixx="0.35498" ixy="0" ixz="0" iyy="0.7266" iyz="0"  izz="1.0553"/>
+      <!-- Moments of inertia: ( chassis without wheels ) -->
+      <inertia
+        ixx="0.35498" ixy="0" ixz="0"
+        iyy="0.7266" iyz="0"
+        izz="1.0553"/>
       </inertial>
   </link>
@@ -116,46 +121,48 @@
       - rear
   -->
-  <link name="front_mount"/>
-  <link name="front_b_mount"/>
-  <link name="front_c_mount"/>
-  <link name="rear_mount"/>
-  <link name="rear_b_mount"/>
-  <link name="rear_c_mount"/>
-  <link name="mid_mount"/>
-  <joint name="mid_mount_joint" type="fixed">
-    <origin xyz="0 0 0.069023" rpy="0 0 0" />
-    <parent link="chassis_link"/>
-    <child link="mid_mount" />
-  </joint>
-  <joint name="front_c_mount_joint" type="fixed">
-    <origin xyz="0.080 0 0" rpy="0 0 0" />
-    <parent link="mid_mount"/>
-    <child link="front_c_mount" />
-  </joint>
-  <joint name="front_b_mount_joint" type="fixed">
-    <origin xyz="0.080 0 0" rpy="0 0 0" />
-    <parent link="front_c_mount"/>
-    <child link="front_b_mount" />
-  </joint>
-  <joint name="front_mount_joint" type="fixed">
-    <origin xyz="0.080 0 0" rpy="0 0 0" />
-    <parent link="front_b_mount"/>
-    <child link="front_mount" />
-  </joint>
-  <joint name="rear_c_mount_joint" type="fixed">
-    <origin xyz="-0.080 0 0" rpy="0 0 0" />
-    <parent link="mid_mount"/>
-    <child link="rear_c_mount" />
-  </joint>
-  <joint name="rear_b_mount_joint" type="fixed">
-    <origin xyz="-0.080 0 0" rpy="0 0 0" />
-    <parent link="rear_c_mount"/>
-    <child link="rear_b_mount" />
-  </joint>
-  <joint name="rear_moint_joint" type="fixed">
-    <origin xyz="-0.080 0 0" rpy="0 0 0" />
-    <parent link="rear_b_mount"/>
-    <child link="rear_mount" />
-  </joint>
+  <xacro:unless value="${pacs_enabled}">
+    <link name="front_mount"/>
+    <link name="front_b_mount"/>
+    <link name="front_c_mount"/>
+    <link name="rear_mount"/>
+    <link name="rear_b_mount"/>
+    <link name="rear_c_mount"/>
+    <link name="mid_mount"/>
+    <joint name="mid_mount_joint" type="fixed">
+      <origin xyz="0 0 0.069023" rpy="0 0 0" />
+      <parent link="chassis_link"/>
+      <child link="mid_mount" />
+    </joint>
+    <joint name="front_c_mount_joint" type="fixed">
+      <origin xyz="0.080 0 0" rpy="0 0 0" />
+      <parent link="mid_mount"/>
+      <child link="front_c_mount" />
+    </joint>
+    <joint name="front_b_mount_joint" type="fixed">
+      <origin xyz="0.080 0 0" rpy="0 0 0" />
+      <parent link="front_c_mount"/>
+      <child link="front_b_mount" />
+    </joint>
+    <joint name="front_mount_joint" type="fixed">
+      <origin xyz="0.080 0 0" rpy="0 0 0" />
+      <parent link="front_b_mount"/>
+      <child link="front_mount" />
+    </joint>
+    <joint name="rear_c_mount_joint" type="fixed">
+      <origin xyz="-0.080 0 0" rpy="0 0 0" />
+      <parent link="mid_mount"/>
+      <child link="rear_c_mount" />
+    </joint>
+    <joint name="rear_b_mount_joint" type="fixed">
+      <origin xyz="-0.080 0 0" rpy="0 0 0" />
+      <parent link="rear_c_mount"/>
+      <child link="rear_b_mount" />
+    </joint>
+    <joint name="rear_moint_joint" type="fixed">
+      <origin xyz="-0.080 0 0" rpy="0 0 0" />
+      <parent link="rear_b_mount"/>
+      <child link="rear_mount" />
+    </joint>
+  </xacro:unless>
   <!--
     Mounting point for accessories on the front bumper.
@@ -169,12 +176,15 @@
     <child link="front_bumper_mount" />
   </joint>
+  <!-- PACS -->
+  <xacro:include filename="$(find arena_simulation_setup)/entities/robots/dingo/urdf/pacs.urdf.xacro"/>
+  <xacro:pacs/>
   <!-- Bring in simulation data for Gazebo. -->
-  <!-- <xacro:include filename="$(find arena_simulation_setup)/entities/robots/dingo/urdf/dingo.gazebo" /> -->
-  <!-- <xacro:include filename="$(find arena_simulation_setup)/entities/robots/dingo/urdf/dingo-o.gazebo" /> -->
+  <xacro:include filename="$(find arena_simulation_setup)/entities/robots/dingo/urdf/dingo.gazebo" />
+  <xacro:include filename="$(find arena_simulation_setup)/entities/robots/dingo/urdf/dingo-o.gazebo" />
   <!-- Optional standard accessories, including their simulation data. The rendering
        of these into the final description is controlled by optenv variables, which
        default each one to off.-->
-  <!-- <xacro:include filename="$(find arena_simulation_setup)/entities/robots/dingo/urdf/accessories.urdf.xacro" /> -->
+  <xacro:include filename="$(find arena_simulation_setup)/entities/robots/dingo/urdf/accessories.urdf.xacro" />
   <!-- Optional custom includes. -->
-  <!-- <xacro:include filename="$(optenv DINGO_URDF_EXTRAS empty.urdf)" /> -->
+  <xacro:include filename="$(optenv DINGO_URDF_EXTRAS empty.urdf)" />
 </robot>
