Commit message: feat(robot): Replace boxer with self-contained package

File: entities/robots/boxer/urdf/boxer.urdf.xacro (robot description, xacro)
@@ -46,5 +46,11 @@
   </gazebo>
   <!-- Lift joint -->
-  <link name="lift_link" />
+  <link name="lift_link">
+    <inertial>
+      <mass value="0.1" />
+      <origin xyz="0 0 0" rpy="0 0 0"/>
+      <inertia ixx="0.001" ixy="0" ixz="0" iyy="0.001" iyz="0" izz="0.001" />
+    </inertial>
+    </link>
   <joint name="lift_joint" type="prismatic">
     <origin rpy="1.5708 0 0" xyz="0 0 0.177"/>

File: entities/robots/boxer/urdf/include/sensors.urdf.xacro (robot description, xacro)
@@ -37,5 +37,5 @@
           <width>640</width>
           <height>480</height>
-          <format>RGB8</format>
+          <format>R8G8B8</format>
         </image>
         <clip>
