Commit message: feat(robot): Replace husky with self-contained package

File: entities/robots/husky/urdf/accessories/flir_blackfly_mount.urdf.xacro (robot description, xacro)
@@ -1,6 +1,6 @@
 <?xml version="1.0"?>
 <robot xmlns:xacro="http://ros.org/wiki/xacro">
-  <xacro:include filename="$(find fath_pivot_mount_description)/urdf/lockmount.urdf.xacro"/>
-  <xacro:include filename="$(find flir_camera_description)/urdf/flir_blackflys.urdf.xacro"/>
+  <xacro:include filename="$(find arena_simulation_setup)/entities/robots/husky/urdf/lockmount.urdf.xacro"/>
+  <xacro:include filename="$(find arena_simulation_setup)/entities/robots/husky/urdf/flir_blackfly_s.urdf.xacro"/>
   <xacro:macro name="flir_blackfly_mount" params="prefix:=blackfly
                                               parent:=top_plate_link
@@ -9,5 +9,5 @@
                                               *origin">
     <!-- Add Blackfly S -->
-    <xacro:flir_blackflys frame="${prefix}"/>
+    <xacro:flir_blackfly_s frame="${prefix}"/>
     <!-- Add Fath Pivot Mouth-->
     <xacro:if value="${mount_enabled}">

File: entities/robots/husky/urdf/accessories/intel_realsense.urdf.xacro (robot description, xacro)
@@ -13,14 +13,14 @@
   '''
   <xacro:if value="${rs_model == 'd435'}">
-    <xacro:include filename="$(find realsense2_description)/urdf/_d435.urdf.xacro" />
+    <xacro:include filename="$(find arena_simulation_setup)/entities/robots/husky/urdf/_d435.urdf.xacro" />
   </xacro:if>
   <xacro:if value="${rs_model == 'd435i'}">
-    <xacro:include filename="$(find realsense2_description)/urdf/_d435i.urdf.xacro" />
+    <xacro:include filename="$(find arena_simulation_setup)/entities/robots/husky/urdf/_d435i.urdf.xacro" />
   </xacro:if>
   <xacro:if value="${rs_model == 'd415'}">
-    <xacro:include filename="$(find realsense2_description)/urdf/_d415.urdf.xacro" />
+    <xacro:include filename="$(find arena_simulation_setup)/entities/robots/husky/urdf/_d415.urdf.xacro" />
   </xacro:if>
   <xacro:if value="${rs_model == 'd455'}">
-    <xacro:include filename="$(find realsense2_description)/urdf/_d435.urdf.xacro" />
+    <xacro:include filename="$(find arena_simulation_setup)/entities/robots/husky/urdf/_d435.urdf.xacro" />
   </xacro:if>
   '''
@@ -43,14 +43,14 @@
     <xacro:if value="${include}">
       <xacro:if value="${rs_model == 'd435'}">
-        <xacro:include filename="$(find realsense2_description)/urdf/_d435.urdf.xacro" />
+        <xacro:include filename="$(find arena_simulation_setup)/entities/robots/husky/urdf/_d435.urdf.xacro" />
       </xacro:if>
       <xacro:if value="${rs_model == 'd435i'}">
-        <xacro:include filename="$(find realsense2_description)/urdf/_d435i.urdf.xacro" />
+        <xacro:include filename="$(find arena_simulation_setup)/entities/robots/husky/urdf/_d435i.urdf.xacro" />
       </xacro:if>
       <xacro:if value="${rs_model == 'd415'}">
-        <xacro:include filename="$(find realsense2_description)/urdf/_d415.urdf.xacro" />
+        <xacro:include filename="$(find arena_simulation_setup)/entities/robots/husky/urdf/_d415.urdf.xacro" />
       </xacro:if>
       <xacro:if value="${rs_model == 'd455'}">
-        <xacro:include filename="$(find realsense2_description)/urdf/_d435.urdf.xacro" />
+        <xacro:include filename="$(find arena_simulation_setup)/entities/robots/husky/urdf/_d435.urdf.xacro" />
       </xacro:if>
     </xacro:if>

File: entities/robots/husky/urdf/accessories/sick_lms1xx_mount.urdf.xacro (robot description, xacro)
@@ -26,5 +26,5 @@
 -->
 <robot xmlns:xacro="http://ros.org/wiki/xacro">
-  <xacro:include filename="$(find lms1xx)/urdf/sick_lms1xx.urdf.xacro" />
+  <xacro:include filename="$(find arena_simulation_setup)/entities/robots/husky/urdf/sick_lms1xx.urdf.xacro" />
   <xacro:macro name="sick_lms1xx_mount" params="prefix parent topic robot_namespace *origin tower:=1">
     <!-- Add SICK LMS1xx -->

File: entities/robots/husky/urdf/accessories/vlp16_mount.urdf.xacro (robot description, xacro)
@@ -1,5 +1,5 @@
 <?xml version="1.0"?>
 <robot xmlns:xacro="http://wiki.ros.org/xacro">
-  <xacro:include filename="$(find velodyne_description)/urdf/VLP-16.urdf.xacro" />
+  <xacro:include filename="$(find arena_simulation_setup)/entities/robots/husky/urdf/VLP-16.urdf.xacro" />
   <xacro:macro name="vlp16_mount" params="prefix parent_link topic height:=0.12 *origin">
     <!--
