Commit message: feat(robot): replace Husky package, clean up RB series meshes & URDF
* Swapped in self-contained Husky (mesh+URDF) under entities/robots/husky
* Removed legacy RBKairos/RBSummit/etc. meshes no longer used
* Added SICK & Hokuyo sensor meshes
* Updated rbrobout URDF to new inertia utils

File: entities/robots/.old/dingo/urdf/accessories.urdf.xacro (robot description, xacro)
@@ -25,6 +25,6 @@
                          topic="$(optenv DINGO_LASER_TOPIC scan)"/> -->
     <xacro:if value="${lidar_model == 'lms1xx'}">
-    <xacro:sick_lms1xx_mount prefix="$(arg robot_namespace)/front"
-                        topic="$(arg robot_namespace)/scan"/>
+    <xacro:sick_lms1xx_mount prefix="$(arg namespace)/front"
+                        topic="$(arg namespace)/scan"/>
       <joint name="$(optenv DINGO_LASER_MOUNT front)_laser_mount_joint" type="fixed">
         <origin xyz="$(optenv DINGO_LASER_OFFSET 0 0 0)"

File: entities/robots/.old/dingo/urdf/dingo.urdf.xacro (robot description, xacro)
@@ -222,5 +222,5 @@
        default each one to off.-->
   <xacro:include filename="$(find arena_simulation_setup)/entities/robots/dingo/urdf/accessories.urdf.xacro" >
-    <xacro:arg name="robot_namespace" value="$(arg robot_namespace)" />
+    <xacro:arg name="robot_namespace" value="$(arg namespace)" />
   </xacro:include>
 </robot>

File: entities/robots/.old/go1/urdf/gazebo.xacro (robot description, xacro)
@@ -5,5 +5,5 @@
     <gazebo>
         <plugin name="gazebo_ros_control" filename="libgazebo_ros_control.so">
-            <robotNamespace>$(arg robot_namespace)</robotNamespace>
+            <robotNamespace>$(arg namespace)</robotNamespace>
             <robotSimType>gazebo_ros_control/DefaultRobotHWSim</robotSimType>
         </plugin>

File: entities/robots/.old/laikago/urdf/gazebo.xacro (robot description, xacro)
@@ -5,5 +5,5 @@
     <gazebo>
         <plugin name="gazebo_ros_control" filename="libgazebo_ros_control.so">
-            <robotNamespace>$(arg robot_namespace)</robotNamespace>
+            <robotNamespace>$(arg namespace)</robotNamespace>
             <robotSimType>gazebo_ros_control/DefaultRobotHWSim</robotSimType>
         </plugin>

File: entities/robots/.old/waffle/urdf/waffle.urdf.xacro (robot description, xacro)
@@ -2,5 +2,5 @@
 <robot name="waffle" xmlns:xacro="http://ros.org/wiki/xacro">
   <xacro:arg name="robot_namespace" default="$(optenv ROBOT_NAMESPACE /)" />
-  <xacro:property name="robot_namespace" value="$(arg robot_namespace)" />
+  <xacro:property name="robot_namespace" value="$(arg namespace)" />
   <xacro:include filename="$(find arena_simulation_setup)/entities/robots/waffle/urdf/common_properties.xacro"/>
   <xacro:include filename="$(find arena_simulation_setup)/entities/robots/waffle/urdf/waffle.gazebo.xacro"/>

File: entities/robots/rbrobout/urdf/all_sensors.urdf.xacro (robot description, xacro)
@@ -1,10 +1,46 @@
 <?xml version="1.0"?>
 <robot name="all_sensors" xmlns:xacro="http://wiki.ros.org/xacro">
-  <!-- Only keep the necessary includes for your sensors -->
-  <!-- 工具宏依赖，部分 sensor 宏可能 include inertia 计算 -->
+  <!-- This file unifies all sensors that can be used on simulation, defined as xacro:macros -->
   <xacro:include filename="$(find arena_simulation_setup)/entities/robots/rbrobout/urdf/utils/inertia.urdf.xacro" />
-  <!-- 2D Lidar Sick Microscan3 -->
+  <!-- Depth sensors -->
+  <xacro:include filename="$(find arena_simulation_setup)/entities/robots/rbrobout/urdf/depth/intel_realsense_d435.urdf.xacro" />
+  <xacro:include filename="$(find arena_simulation_setup)/entities/robots/rbrobout/urdf/depth/intel_realsense_d435i.urdf.xacro" />
+  <xacro:include filename="$(find arena_simulation_setup)/entities/robots/rbrobout/urdf/depth/orbbec_astra.urdf.xacro" />
+  <xacro:include filename="$(find arena_simulation_setup)/entities/robots/rbrobout/urdf/depth/stereolabs_generic.urdf.xacro" />
+  <xacro:include filename="$(find arena_simulation_setup)/entities/robots/rbrobout/urdf/depth/stereolabs_zed2.urdf.xacro" />
+  <xacro:include filename="$(find arena_simulation_setup)/entities/robots/rbrobout/urdf/depth/stereolabs_zed2i.urdf.xacro" />
+  <xacro:include filename="$(find arena_simulation_setup)/entities/robots/rbrobout/urdf/depth/azure_kinect.urdf.xacro" />
+  <!-- 2D Lidars -->
   <xacro:include filename="$(find arena_simulation_setup)/entities/robots/rbrobout/urdf/2d_lidar/sick_microscan3.urdf.xacro" />
-  <!-- IMU Vectornav -->
+  <xacro:include filename="$(find arena_simulation_setup)/entities/robots/rbrobout/urdf/2d_lidar/sick_nanoscan3.urdf.xacro" />
+  <xacro:include filename="$(find arena_simulation_setup)/entities/robots/rbrobout/urdf/2d_lidar/sick_outdoorscan3.urdf.xacro" />
+  <xacro:include filename="$(find arena_simulation_setup)/entities/robots/rbrobout/urdf/2d_lidar/sick_s300.urdf.xacro" />
+  <xacro:include filename="$(find arena_simulation_setup)/entities/robots/rbrobout/urdf/2d_lidar/sick_s3000.urdf.xacro" />
+  <xacro:include filename="$(find arena_simulation_setup)/entities/robots/rbrobout/urdf/2d_lidar/sick_tim551.urdf.xacro" />
+  <xacro:include filename="$(find arena_simulation_setup)/entities/robots/rbrobout/urdf/2d_lidar/sick_tim571.urdf.xacro" />
+  <xacro:include filename="$(find arena_simulation_setup)/entities/robots/rbrobout/urdf/2d_lidar/hokuyo_urg04lx.urdf.xacro" />
+  <xacro:include filename="$(find arena_simulation_setup)/entities/robots/rbrobout/urdf/2d_lidar/hokuyo_ust10lx.urdf.xacro" />
+  <xacro:include filename="$(find arena_simulation_setup)/entities/robots/rbrobout/urdf/2d_lidar/hokuyo_ust20lx.urdf.xacro" />
+  <xacro:include filename="$(find arena_simulation_setup)/entities/robots/rbrobout/urdf/2d_lidar/hokuyo_utm30lx.urdf.xacro" />
+  <!-- 3D Lidars -->
+  <xacro:include filename="$(find arena_simulation_setup)/entities/robots/rbrobout/urdf/3d_lidar/velodyne_vlp16.urdf.xacro" />
+  <xacro:include filename="$(find arena_simulation_setup)/entities/robots/rbrobout/urdf/3d_lidar/robosense_bpearl.urdf.xacro" />
+  <xacro:include filename="$(find arena_simulation_setup)/entities/robots/rbrobout/urdf/3d_lidar/robosense_helios_16p.urdf.xacro" />
+  <xacro:include filename="$(find arena_simulation_setup)/entities/robots/rbrobout/urdf/3d_lidar/ouster.urdf.xacro" />
+  <xacro:include filename="$(find arena_simulation_setup)/entities/robots/rbrobout/urdf/3d_lidar/livox_mid_360.urdf.xacro" />
+  <xacro:include filename="$(find arena_simulation_setup)/entities/robots/rbrobout/urdf/3d_lidar/sick_multiscan_100.urdf.xacro" />
+  <!-- IMUs -->
   <xacro:include filename="$(find arena_simulation_setup)/entities/robots/rbrobout/urdf/imu/vectornav.urdf.xacro" />
+  <xacro:include filename="$(find arena_simulation_setup)/entities/robots/rbrobout/urdf/imu/myahrs.urdf.xacro" />
+  <xacro:include filename="$(find arena_simulation_setup)/entities/robots/rbrobout/urdf/imu/pixhawk.urdf.xacro" />
+  <!-- GPS -->
+  <xacro:include filename="$(find arena_simulation_setup)/entities/robots/rbrobout/urdf/gps/gps.urdf.xacro" />
+  <xacro:include filename="$(find arena_simulation_setup)/entities/robots/rbrobout/urdf/gps/gps_with_mast.urdf.xacro" />
+  <xacro:include filename="$(find arena_simulation_setup)/entities/robots/rbrobout/urdf/gps/ublox.urdf.xacro" />
+  <xacro:include filename="$(find arena_simulation_setup)/entities/robots/rbrobout/urdf/gps/ublox_with_mast.urdf.xacro" />
+  <!-- Camera -->
+  <xacro:include filename="$(find arena_simulation_setup)/entities/robots/rbrobout/urdf/camera/axis_m5013.urdf.xacro" />
+  <xacro:include filename="$(find arena_simulation_setup)/entities/robots/rbrobout/urdf/camera/axis_m5074.urdf.xacro" />
+  <xacro:include filename="$(find arena_simulation_setup)/entities/robots/rbrobout/urdf/camera/axis_m5525.urdf.xacro" />
+  <xacro:include filename="$(find arena_simulation_setup)/entities/robots/rbrobout/urdf/camera/axis_m5526.urdf.xacro" />
 </robot>

File: entities/robots/rbrobout/urdf/bases/rbrobout/rbrobout_base.urdf.xacro (robot description, xacro)
@@ -10,5 +10,5 @@
   	<xacro:include filename="$(find arena_simulation_setup)/entities/robots/rbrobout/urdf/wheels/mecanum_wheel/rbrobout_mecanum_wheel.urdf.xacro" />
 	<!-- Import all available sensors -->
-	<xacro:include filename="$(find robotnik_sensors)/urdf/all_sensors.urdf.xacro" />
+	<xacro:include filename="$(find arena_simulation_setup)/entities/robots/rbrobout/urdf/all_sensors.urdf.xacro" />
 	<xacro:property name="PI" value="3.1415926535897931"/>
 	<!-- Wheel parameters -->

File: entities/robots/rbrobout/urdf/rbrobout.urdf.xacro (robot description, xacro)
@@ -1,42 +1,69 @@
-<robot name="rbrobout" xmlns:xacro="http://www.ros.org/wiki/xacro">
-  <link name="base_link"/>
+<?xml version="1.0"?>
+<robot name="rbrobout" xmlns:xacro="http://wiki.ros.org/xacro">
+  <!-- ***************** -->
+  <!-- Imported elements -->
+  <!-- ***************** -->
+  <!-- Import all posible elements defined in the urdf.xacro files. All these elements are defined as macro:xacros -->
+  <xacro:include filename="$(find arena_simulation_setup)/entities/robots/rbrobout/urdf/bases/rbrobout/rbrobout_base.urdf.xacro" />
+  <xacro:include filename="$(find arena_simulation_setup)/entities/robots/rbrobout/urdf/base_hw/rbrobout.ros2_control.urdf" />
+  <xacro:include filename="$(find arena_simulation_setup)/entities/robots/rbrobout/simulators/gazebo_classic/rbrobout/rbrobout_control.urdf.xacro" />
+  <xacro:include filename="$(find arena_simulation_setup)/entities/robots/rbrobout/simulators/gazebo_ignition/rbrobout/rbrobout_control.urdf.xacro" />
+  <xacro:include filename="$(find arena_simulation_setup)/entities/robots/rbrobout/urdf/all_sensors.urdf.xacro" />
+  <!-- Properties and Arguments -->
+  <xacro:arg name="namespace" default="robot"/>
+  <xacro:arg name="prefix" default="robot_"/>
+  <xacro:arg name="gazebo_classic" default="false"/>
+  <xacro:arg name="gazebo_ignition" default="false"/>
+  <xacro:property name="front_laser_offset_x" value="0.8"/>
+  <xacro:property name="front_laser_offset_y" value="0.366"/>
+  <xacro:property name="front_laser_offset_z" value="-0.06"/>
+  <xacro:property name="rear_laser_offset_x" value="-0.8"/>
+  <xacro:property name="rear_laser_offset_y" value="-0.366"/>
+  <xacro:property name="rear_laser_offset_z" value="-0.06"/>
+  <xacro:property name="imu_offset_x" value="0.3"/>
+  <xacro:property name="imu_offset_y" value="-0.3"/>
+  <xacro:property name="imu_offset_z" value="0.0725"/>
+  <xacro:rbrobout prefix="$(arg prefix)" gazebo_classic="$(arg gazebo_classic)" gazebo_ignition="$(arg gazebo_ignition)"/>
   <!-- IMU -->
-  <link name="imu_link">
-    <inertial>
-      <mass value="0.001"/>
-      <origin xyz="0 0 0" rpy="0 0 0"/>
-      <inertia ixx="1e-9" ixy="0.0" ixz="0.0" iyy="1e-9" iyz="0.0" izz="1e-9"/>
-    </inertial>
-  </link>
-  <joint name="imu_joint" type="fixed">
-    <parent link="base_link"/>
-    <child link="imu_link"/>
-    <origin xyz="0.0 0.0 0.10"/>
-  </joint>
-  <!-- LiDAR -->
-  <link name="lidar_link">
-    <visual>
-      <geometry>
-        <cylinder radius="0.05" length="0.1"/>
-      </geometry>
-      <origin xyz="0 0 0"/>
-      <material name="black"/>
-    </visual>
-    <collision>
-      <geometry>
-        <cylinder radius="0.05" length="0.1"/>
-      </geometry>
-      <origin xyz="0 0 0"/>
-    </collision>
-    <inertial>
-      <origin xyz="0 0 0"/>
-      <mass value="0.1"/>
-      <inertia ixx="1e-5" ixy="0" ixz="0" iyy="1e-5" iyz="0" izz="1e-5"/>
-    </inertial>
-  </link>
-  <joint name="lidar_joint" type="fixed">
-    <parent link="base_link"/>
-    <child link="lidar_link"/>
-    <origin xyz="0.0 0.0 0.2"/>
-  </joint>
+    <xacro:sensor_vectornav
+        frame_prefix="$(arg prefix)vectornav_"
+        parent="$(arg prefix)base_link"
+        node_namespace="$(arg namespace)"
+        gazebo_classic="$(arg gazebo_classic)"
+        gazebo_ignition="$(arg gazebo_ignition)">
+        <origin xyz="${imu_offset_x} ${imu_offset_y} ${imu_offset_z}" rpy="0 0 0"/>
+    </xacro:sensor_vectornav>
+  <!-- 2d laser -->
+    <xacro:sensor_sick_microscan3
+        frame_prefix="$(arg prefix)front_laser_"
+        parent="$(arg prefix)base_link"
+        node_namespace="$(arg namespace)"
+        node_name="front_laser"
+        gazebo_classic="$(arg gazebo_classic)"
+        gazebo_ignition="$(arg gazebo_ignition)">
+        <origin xyz="${front_laser_offset_x} ${front_laser_offset_y} ${front_laser_offset_z}" rpy="0 0 ${1/4*PI}"/>
+    </xacro:sensor_sick_microscan3>
+    <!-- 2d laser -->
+    <xacro:sensor_sick_microscan3
+        frame_prefix="$(arg prefix)rear_laser_"
+        parent="$(arg prefix)base_link"
+        node_namespace="$(arg namespace)"
+        node_name="rear_laser"
+        gazebo_classic="$(arg gazebo_classic)"
+        gazebo_ignition="$(arg gazebo_ignition)">
+        <origin xyz="${rear_laser_offset_x} ${rear_laser_offset_y} ${rear_laser_offset_z}" rpy="0 0 ${-3/4*PI}"/>
+    </xacro:sensor_sick_microscan3>
+    <!-- Controllers -->
+    <xacro:if value="$(arg gazebo_classic)">
+        <xacro:rbrobout_gz_classic_control namespace="$(arg namespace)" prefix="$(arg prefix)"/>
+        <xacro:ros_planar_move_gazebo_classic/>
+    </xacro:if>
+    <xacro:if value="$(arg gazebo_ignition)">
+        <xacro:rbrobout_gz_ignition_control namespace="$(arg namespace)" prefix="$(arg prefix)"/>
+    </xacro:if>
+    <xacro:unless value="$(arg gazebo_classic)">
+        <xacro:unless value="$(arg gazebo_ignition)">
+            <xacro:rbrobout_base_hw_controller/>
+        </xacro:unless>
+    </xacro:unless>
 </robot>

File: entities/robots/rbrobout/urdf/utils/inertia.urdf.xacro (robot description, xacro)
@@ -10,5 +10,5 @@
   </xacro:macro>
   <!-- TODO Hollow sphere of radius r and mass m-->
-  <xacro:macro name="hollow_sphere_inertia" params="m r">
+  <xacro:macro name="solid_sphere_inertia" params="m r">
     <inertia  ixx="${(2*r*r*m)/3}" ixy = "0" ixz = "0"
               iyy="${(2*r*r*m)/3}" iyz = "0"
@@ -16,8 +16,22 @@
      />
   </xacro:macro>
+  <!-- TODO Solid ellipsoid of semi-axes a, b, c and mass m-->
+  <xacro:macro name="ellipsoid_semi_axes_inertia" params="a b c m r">
+    <inertia  ixx="${(m*(b*b+c*c))/5}" ixy = "0" ixz = "0"
+              iyy="${(m*(a*a+c*c))/5}" iyz = "0"
+              izz="${(m*(a*a+b*b))/5}"
+     />
+  </xacro:macro>
+  <!-- TODO Right circular cone with radius r, height h and mass m, about the apex -->
+  <xacro:macro name="right_circular_cone_inertia" params="m r h">
+    <inertia  ixx="${((3*m*(h*h))/5)+((3*m*(r*r))/20)}" ixy = "0" ixz = "0"
+              iyy="${((3*m*(h*h))/5)+((3*m*(r*r))/20)}" iyz = "0"
+              izz="${(3*m*(r*r))/10}"
+     />
+  </xacro:macro>
   <!-- TODO Solid cuboid of width w, height h, depth d, and mass m -->
-  <!-- yes, axis in solid_cuboid_inertia are changed, w relates to X axis, d to Z axis, and h to Y axis -->
+  <!-- w relates to X axis, d to Z axis, and h to Y axis -->
   <!-- Keep this comment -->
-  <xacro:macro name="solid_cuboid_inertia" params="m h d w">
+  <xacro:macro name="solid_cuboid_inertia" params="m w h d">
     <inertia  ixx="${(m*(h*h+d*d))/12}" ixy = "0" ixz = "0"
               iyy="${(m*(w*w+d*d))/12}" iyz = "0"
@@ -32,3 +46,10 @@
      />
   </xacro:macro>
+    <!-- TODO Thick-walled cylindrical tube with open ends, of inner radius r1, outer radius r2, length h and mass m -->
+    <xacro:macro name="thick_walled_cylinder_inertia" params="m r1 r2 h">
+    <inertia  ixx="${m*((3*(r1*r1+r2*r2))+(h*h))/12}" ixy = "0" ixz = "0"
+              iyy="${m*((3*(r1*r1+r2*r2))+(h*h))/12}" iyz = "0"
+              izz="${m*(r1*r1+r2*r2)/2}"
+     />
+  </xacro:macro>
 </robot>
