Commit message: feat(robot): Replace rb with self-contained package

File: entities/robots/dingo/urdf/accessories/hokuyo_ust10.urdf.xacro (robot description, xacro)
@@ -15,5 +15,6 @@
       <gazebo reference="${frame}">
         <turnGravityOff>true</turnGravityOff>
-        <sensor type="ray" name="${frame}">
+        <sensor type="gpu_lidar" name="${frame}">
+          <gz_frame_id>dingo/front_laser</gz_frame_id>
           <pose>0 0 0 0 0 0</pose>
           <visualize>false</visualize>

File: entities/robots/dingo/urdf/accessories/intel_realsense.urdf.xacro (robot description, xacro)
@@ -86,5 +86,5 @@
              <height>${height}</height>
              <!-- TODO: check what format the Realsense hardware delivers and set this to match! -->
-             <format>RGB8</format>
+             <format>R8G8B8</format>
            </image>
            <clip>

File: entities/robots/rbkairos/simulators/gazebo_classic/rbkairos/rbkairos_control.urdf.xacro (robot description, xacro)
@@ -3,5 +3,5 @@
     <xacro:macro name="rbkairos_gz_classic_control"  params="namespace prefix">
         <gazebo>
-          <plugin name="ros_control" filename="libgazebo_ros2_control.so">
+          <!-- <plugin name="ros_control" filename="libgazebo_ros2_control.so">
             <robot_param>robot_description</robot_param>
             <robot_param_node>robot_state_publisher</robot_param_node>
@@ -10,4 +10,16 @@
                 <namespace>/${namespace}</namespace>
             </ros>
+          </plugin> -->
+          <plugin filename="gz-sim-diff-drive-system" name="gz::sim::systems::DiffDrive">
+            <left_joint>robot_back_left_wheel_joint</left_joint>
+            <right_joint>robot_front_right_wheel_joint</right_joint>
+            <left_joint>robot_front_left_wheel_joint</left_joint>
+            <right_joint>robot_back_right_wheel_joint</right_joint>
+            <wheel_separation>0.48</wheel_separation>
+            <wheel_radius>0.095</wheel_radius>
+            <odom_publish_frequency>50</odom_publish_frequency>
+            <publish_odom>true</publish_odom>
+            <publish_odom_tf>true</publish_odom_tf>
+            <publish_wheel_tf>true</publish_wheel_tf>
           </plugin>
         </gazebo>

File: entities/robots/rbkairos/simulators/gazebo_ignition/rbkairos/rbkairos_control.urdf.xacro (robot description, xacro)
@@ -3,5 +3,5 @@
   <xacro:macro name="rbkairos_gz_ignition_control"  params="namespace prefix">
       <gazebo>
-        <plugin name="gz_ros2_control::GazeboSimROS2ControlPlugin" filename="gz_ros2_control-system">
+        <!-- <plugin name="gz_ros2_control::GazeboSimROS2ControlPlugin" filename="gz_ros2_control-system">
           <robot_param>robot_description</robot_param>
           <robot_param_node>robot_state_publisher</robot_param_node>
@@ -10,4 +10,19 @@
               <namespace>/${namespace}</namespace>
           </ros>
+        </plugin> -->
+        <plugin filename="gz-sim-diff-drive-system" name="gz::sim::systems::DiffDrive">
+          <left_joint>robot_back_left_wheel_joint</left_joint>
+          <right_joint>robot_front_right_wheel_joint</right_joint>
+          <left_joint>robot_front_left_wheel_joint</left_joint>
+          <right_joint>robot_back_right_wheel_joint</right_joint>
+          <!-- <wheel_separation>0.48</wheel_separation>
+          <wheel_radius>0.095</wheel_radius>
+          <odom_publish_frequency>50</odom_publish_frequency> -->
+          <wheel_separation>0.70</wheel_separation>
+          <wheel_radius>0.10</wheel_radius>
+          <odom_publish_frequency>50</odom_publish_frequency>
+          <publish_odom>true</publish_odom>
+          <publish_odom_tf>true</publish_odom_tf>
+          <publish_wheel_tf>true</publish_wheel_tf>
         </plugin>
       </gazebo>
@@ -23,5 +38,5 @@
         </joint>
       </xacro:macro>
-      <ros2_control name="IgnitionSystem" type="system">
+      <!-- <ros2_control name="IgnitionSystem" type="system">
         <hardware>
             <plugin>gz_ros2_control/GazeboSimSystem</plugin>
@@ -31,5 +46,5 @@
         <xacro:ros2_joint interface="velocity" jmin="-20" jmax="20" name="${prefix}back_left_wheel_joint"/>
         <xacro:ros2_joint interface="velocity" jmin="-20" jmax="20" name="${prefix}back_right_wheel_joint"/>
-      </ros2_control>
+      </ros2_control> -->
   </xacro:macro>
 </robot>

File: entities/robots/rbkairos/urdf/2d_lidar/lidar_2d_plugin.urdf.xacro (robot description, xacro)
@@ -15,7 +15,8 @@
             samples
             ">
-    <xacro:if value="${gazebo_classic}">
+    <!-- <xacro:if value="${gazebo_classic}">
       <gazebo reference="${frame_link}">
-        <sensor type="ray" name="${frame_prefix}sensor">
+        <sensor type="gpu_lidar" name="${frame_prefix}sensor">
+          <gz_frame_id>$(arg name)/${frame_prefix}sensor</gz_frame_id>
           <pose>0 0 0 0 0 0</pose>
           <visualize>false</visualize>
@@ -53,8 +54,9 @@
         </sensor>
       </gazebo>
-    </xacro:if>
-    <xacro:if value="${gazebo_ignition}">
+    </xacro:if> -->
+    <!-- <xacro:if value="${gazebo_ignition}"> -->
       <gazebo reference="${frame_link}">
         <sensor type="gpu_lidar" name="${node_name}">
+          <gz_frame_id>$(arg name)/${node_name}</gz_frame_id>
           <pose>0 0 0 0 0 0</pose>
           <visualize>false</visualize>
@@ -84,5 +86,55 @@
         </sensor>
       </gazebo>
-    </xacro:if>
+    <!-- </xacro:if> -->
   </xacro:macro>
 </robot>
+<!-- <?xml version="1.0"?>
+<robot name="lidar_2d_plugin" xmlns:xacro="http://wiki.ros.org/xacro">
+  <xacro:macro name="lidar_2d_plugin" params="
+            node_namespace
+            node_name
+            gazebo_classic
+            gazebo_ignition
+            min_range
+            max_range
+            min_angle
+            max_angle
+            frame_link
+            rate
+            resolution
+            samples
+            ">
+    <gazebo reference="${frame_link}">
+        <sensor type="gpu_lidar" name="${node_name}_sensor">
+          <pose>0 0 0 0 0 0</pose>
+          <visualize>false</visualize>
+          <update_rate>${rate}</update_rate>
+          <ray>
+            <scan>
+              <horizontal>
+                <samples>${samples}</samples>
+                <resolution>1</resolution>
+                <min_angle>${min_angle}</min_angle>
+                <max_angle>${max_angle}</max_angle>
+              </horizontal>
+            </scan>
+            <range>
+              <min>${min_range}</min>
+              <max>${max_range}</max>
+              <resolution>0.01</resolution>
+            </range>
+             <noise>
+              <type>gaussian</type>
+              <mean>0.0</mean>
+              <stddev>0.01</stddev>
+            </noise>
+          </ray>
+          <plugin name="gazebo_ros_laser" filename="libgazebo_ros_laser.so">
+            <topicName>${node_name}</topicName>
+            <frameName>${frame_link}</frameName>
+            <robotNamespace>${node_namespace}</robotNamespace>
+          </plugin>
+        </sensor>
+    </gazebo>
+  </xacro:macro>
+</robot> -->

File: entities/robots/rbkairos/urdf/2d_lidar/sick_outdoorscan3.urdf.xacro (robot description, xacro)
@@ -70,5 +70,6 @@
     </xacro:unless>
       <gazebo reference="${frame_prefix}link">
-        <sensor type="${ray_type}" name="${frame_prefix}sensor">
+        <sensor type="gpu_lidar" name="${frame_prefix}sensor">
+          <gz_frame_id>$(arg name)/${frame_prefix}sensor</gz_frame_id>
           <pose>0.0 0.0 0.0 0.0 0.0 0.0</pose>
           <visualize>false</visualize>

File: entities/robots/rbkairos/urdf/3d_lidar/lidar_3d_plugin.urdf.xacro (robot description, xacro)
@@ -17,5 +17,6 @@
     <xacro:if value="${gazebo_classic}">
     <gazebo reference="${frame_link}">
-        <sensor type="ray" name="${node_name}">
+        <sensor type="gpu_lidar" name="${node_name}">
+          <gz_frame_id>$(arg name)/${node_name}</gz_frame_id>
           <pose>0 0 0 0 0 0</pose>
           <visualize>false</visualize>
@@ -62,4 +63,5 @@
       <gazebo reference="${frame_link}">
         <sensor type="gpu_lidar" name="${node_name}">
+          <gz_frame_id>$(arg name)/${node_name}</gz_frame_id>
           <pose>0 0 0 0 0 0</pose>
           <visualize>false</visualize>

File: entities/robots/rbkairos/urdf/camera/camera_plugin.urdf.xacro (robot description, xacro)
@@ -17,5 +17,5 @@
             rate
             ">
-    <xacro:if value="${gazebo_classic}">
+    <!-- <xacro:if value="${gazebo_classic}">
       <gazebo reference="${reference_frame}">
         <sensor name="${node_name}" type="camera">
@@ -50,6 +50,6 @@
         </sensor>
       </gazebo>
-    </xacro:if>
-    <xacro:if value="${gazebo_ignition}">
+    </xacro:if> -->
+    <!-- <xacro:if value="${gazebo_ignition}"> -->
       <gazebo reference="${reference_frame}">
         <sensor name="${node_name}" type="camera">
@@ -80,5 +80,5 @@
         </sensor>
       </gazebo>
-    </xacro:if>
+    <!-- </xacro:if> -->
   </xacro:macro>
 </robot>

File: entities/robots/rbkairos/urdf/deprecated/asus_xtion_pro.urdf.xacro (robot description, xacro)
@@ -104,4 +104,5 @@
     <gazebo reference="${frame_prefix}depth_link">
       <sensor type="depth" name="${node_name}sensor">
+        <gz_frame_id>$(arg name)/${node_name}sensor</gz_frame_id>
         <always_on>true</always_on>
         <update_rate>20.0</update_rate>

File: entities/robots/rbkairos/urdf/deprecated/axis.urdf.xacro (robot description, xacro)
@@ -122,4 +122,5 @@
     <gazebo reference="${prefix}_frame_link">
       <sensor type="camera" name="${prefix}_sensor">
+        <gz_frame_id>$(arg name)/${prefix}_sensor</gz_frame_id>
         <update_rate>30.0</update_rate>
         <camera>

File: entities/robots/rbkairos/urdf/deprecated/axis_q8641.urdf.xacro (robot description, xacro)
@@ -168,4 +168,5 @@
     <gazebo reference="${prefix}_frame_link">
       <sensor type="camera" name="${prefix}_sensor">
+        <gz_frame_id>$(arg name)/${prefix}_sensor</gz_frame_id>
         <update_rate>30.0</update_rate>
         <camera>

File: entities/robots/rbkairos/urdf/deprecated/benewake_ce30.urdf.xacro (robot description, xacro)
@@ -52,5 +52,6 @@
         <xacro:property name="plugin_lib" value="libgazebo_ros_velodyne_laser.so" />
       </xacro:unless>
-        <sensor type="${ray_type}" name="${prefix}_sensor">
+        <sensor type="gpu_lidar" name="${prefix}_sensor">
+          <gz_frame_id>$(arg name)/${prefix}_sensor</gz_frame_id>
           <pose>0 0 0 0 0 0.0</pose>
           <visualize>false</visualize>

File: entities/robots/rbkairos/urdf/deprecated/benewake_ce30d.urdf.xacro (robot description, xacro)
@@ -53,5 +53,6 @@
         <xacro:property name="plugin_lib" value="libgazebo_ros_block_laser.so" />
       </xacro:unless>
-        <sensor type="${ray_type}" name="${prefix}_sensor">
+        <sensor type="gpu_lidar" name="${prefix}_sensor">
+          <gz_frame_id>$(arg name)/${prefix}_sensor</gz_frame_id>
           <pose>0 0 0 0 0 0.0</pose>
           <visualize>false</visualize>

File: entities/robots/rbkairos/urdf/deprecated/embedded_s.urdf.xacro (robot description, xacro)
@@ -64,4 +64,5 @@
     <gazebo reference="${prefix}_link">
       <sensor type="depth" name="${prefix}_depth_sensor">
+        <gz_frame_id>$(arg name)/${prefix}_depth_sensor</gz_frame_id>
         <always_on>true</always_on>
         <update_rate>20.0</update_rate>

File: entities/robots/rbkairos/urdf/deprecated/fotonic_e.urdf.xacro (robot description, xacro)
@@ -62,4 +62,5 @@
     <gazebo reference="${prefix}_depth_frame_link">
       <sensor type="depth" name="${prefix}_sensor">
+        <gz_frame_id>$(arg name)/${prefix}_sensor</gz_frame_id>
         <update_rate>30.0</update_rate>
         <camera name="fotonic">

File: entities/robots/rbkairos/urdf/deprecated/hokuyo3d.urdf.xacro (robot description, xacro)
@@ -47,5 +47,6 @@
         <xacro:property name="plugin_lib" value="libgazebo_ros_velodyne_laser.so" />
       </xacro:unless>
-      <sensor type="${ray_type}" name="${prefix}_sensor">
+      <sensor type="gpu_lidar" name="${prefix}_sensor">
+        <gz_frame_id>$(arg name)/${prefix}_sensor</gz_frame_id>
           <pose>0 0 0 0 0 0</pose>
           <visualize>false</visualize>

File: entities/robots/rbkairos/urdf/deprecated/intel_r430.urdf.xacro (robot description, xacro)
@@ -109,4 +109,5 @@
     <gazebo reference="${prefix}_camera_link">
       <sensor type="depth" name="${prefix}_depth_sensor">
+        <gz_frame_id>$(arg name)/${prefix}_depth_sensor</gz_frame_id>
         <always_on>true</always_on>
         <update_rate>15.0</update_rate>

File: entities/robots/rbkairos/urdf/deprecated/kinect.urdf.xacro (robot description, xacro)
@@ -70,4 +70,5 @@
     <gazebo reference="${prefix}_link">
       <sensor type="depth" name="${prefix}_sensor">
+        <gz_frame_id>$(arg name)/${prefix}_sensor</gz_frame_id>
         <always_on>true</always_on>
         <update_rate>20.0</update_rate>

File: entities/robots/rbkairos/urdf/deprecated/kinectv2.urdf.xacro (robot description, xacro)
@@ -90,4 +90,5 @@
     <gazebo reference="${prefix}_link">
       <sensor type="depth" name="${prefix}_sensor">
+        <gz_frame_id>$(arg name)/${prefix}_sensor</gz_frame_id>
         <always_on>true</always_on>
         <update_rate>20.0</update_rate>

File: entities/robots/rbkairos/urdf/deprecated/pointgrey_bumblebee2.urdf.xacro (robot description, xacro)
@@ -5,4 +5,5 @@
     <gazebo reference="${prefix}_frame">
       <sensor type="multicamera" name="stereo_camera">
+        <gz_frame_id>$(arg name)/stereo_camera</gz_frame_id>
         <update_rate>${fps}</update_rate>
         <camera name="left">
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